File: pcb/fast-pwm.sch (KiCad schematic (older format))
At the start: 42 parts, among them J1 Conn_01x13_Female, J2 Клемма питания, J3 Выходная клемма, J4 Conn_01x02_Male, Q1 2N3904, Q10 AOD4184A, Q11 AOD4184A, Q12 AOD4184A, Q2 2N3905, Q3 2N3904, Q4 2N3905, Q5 2N3904, Q6 2N3905, Q7 2N3904, Q8 2N3905, Q9 AOD4184A, U1 STM32F030K6Tx, U2 MC33063AD

Commit message: версия 0.3
Parts:
- removed J1: Conn_01x13_Female, Connector_PinHeader_2.54mm:PinHeader_1x13_P2.54mm_Vertical, symbol Connector:Conn_01x13_Female
- removed J4: Conn_01x02_Male, Connector_PinHeader_2.54mm:PinHeader_1x02_P2.54mm_Vertical, symbol Connector:Conn_01x02_Male
- added J1: SWD, Connector_PinHeader_2.54mm:PinHeader_1x02_P2.54mm_Vertical, symbol Connector:Conn_01x02_Female
- added J4: ENC1, Connector_JST:JST_ZE_BM04B-ZESS-TBT_1x04-1MP_P1.50mm_Vertical, symbol Connector:Conn_01x04_Female
- added J5: I2C, Connector_JST:JST_ZE_BM04B-ZESS-TBT_1x04-1MP_P1.50mm_Vertical, symbol Connector:Conn_01x04_Female
- added J6: UART, Connector_JST:JST_ZE_BM04B-ZESS-TBT_1x04-1MP_P1.50mm_Vertical, symbol Connector:Conn_01x04_Female
Connections:
- net labels added: CURRENT_CH1, CURRENT_CH2, CURRENT_CH3, CURRENT_CH4
- net labels removed: LED_BLUE, LED_GREEN, LED_RED, SEG1, SEG2, SEG3, SEG4, SEG5, SEG6, SEG7
Other:
- moved on the sheet: R13, R14
